Commit message: omni wheel urdf edittd

File: summit/summit_xl_description/robots/summit_xl_omni.urdf (robot description, URDF)
Before this commit: robot summit_xl, 22 links, 21 joints
Links:
- link summit_xl_back_left_wheel_link: geometry collision mesh filename=package://summit_xl_description/meshes/wheels/omni_wheel_1.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; visual mesh filename=package://summit_xl_description/meshes/wheels/omni_wheel_1.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
- link summit_xl_back_right_wheel_link: geometry collision mesh filename=package://summit_xl_description/meshes/wheels/omni_wheel_2.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; visual mesh filename=package://summit_xl_description/meshes/wheels/omni_wheel_2.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
- link summit_xl_front_left_wheel_link: geometry collision mesh filename=package://summit_xl_description/meshes/wheels/omni_wheel_1.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; visual mesh filename=package://summit_xl_description/meshes/wheels/omni_wheel_1.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
- link summit_xl_front_right_wheel_link: geometry collision mesh filename=package://summit_xl_description/meshes/wheels/omni_wheel_2.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; visual mesh filename=package://summit_xl_description/meshes/wheels/omni_wheel_2.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

File: summit/summit_xl_description/robots/summit_xl_omni.urdf.xacro (robot description, xacro)
@@ -54,8 +54,8 @@
   			<origin xyz="${wheel_offset_x} ${wheel_offset_y} ${wheel_offset_z}" rpy="0 0 0"/>
   		</xacro:omni_wheel>
-  		<xacro:omni_wheel prefix="$(arg prefix)back_left" parent="$(arg prefix)base_link" reflect="true" hq="${hq}">
+  		<xacro:omni_wheel prefix="$(arg prefix)back_left" parent="$(arg prefix)base_link" reflect="false" hq="${hq}">
   			<origin xyz="-${wheel_offset_x} ${wheel_offset_y} ${wheel_offset_z}" rpy="0 0 0"/>
   		</xacro:omni_wheel>
-  		<xacro:omni_wheel prefix="$(arg prefix)back_right" parent="$(arg prefix)base_link" reflect="false" hq="${hq}">
+  		<xacro:omni_wheel prefix="$(arg prefix)back_right" parent="$(arg prefix)base_link" reflect="true" hq="${hq}">
   			<origin xyz="-${wheel_offset_x} -${wheel_offset_y} ${wheel_offset_z}" rpy="0 0 0"/>
   		</xacro:omni_wheel>

File: summit/summit_xl_description/urdf/wheels/omni_wheel.urdf.xacro (robot description, xacro)
@@ -46,5 +46,5 @@
       </visual>
       <collision>
-				<origin xyz="0 0 0" rpy="${PI/2} 0 0" />
+				<origin xyz="0 0 0" rpy="0 0 0" />
         <geometry>
           <xacro:if value="${reflect}">

Commit message: for video shooting

File: summit/summit_xl_description/robots/summit_xl_omni.urdf (robot description, URDF)
Before this commit: robot summit_xl, 22 links, 21 joints
Links:
- link summit_xl_back_left_wheel_link: geometry collision mesh filename=package://summit_xl_description/meshes/wheels/omni_wheel_2.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; visual mesh filename=package://summit_xl_description/meshes/wheels/omni_wheel_2.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
- link summit_xl_back_right_wheel_link: geometry collision mesh filename=package://summit_xl_description/meshes/wheels/omni_wheel_1.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; visual mesh filename=package://summit_xl_description/meshes/wheels/omni_wheel_1.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
