Commit message: thin urdf with cam

File: limo_description/urdf/limo_diff_thin.urdf (robot description, URDF)
Before this commit: robot limo_diffferential, 7 links, 6 joints
Links:
- added link depth_camera_link, mass 0.1; collision box size=0.02 0.06 0.015; visual box size=0.02 0.06 0.015
- added link depth_link
- added link imu_link, mass 0.01; collision box size=0.001 0.001 0.001; visual box size=0.001 0.001 0.001
- added link laser_link, mass 0.1; collision cylinder length=0.016 radius=0.032; visual cylinder length=0.01 radius=0.02
Joints:
- added joint depth_camera_joint: type fixed, parent base_link, child depth_camera_link, origin xyz=0.084 0 0.03 rpy=0 0 0
- added joint depth_camera_to_camera_joint: type fixed, parent depth_camera_link, child depth_link, origin xyz=0 0 0 rpy=-1.57 0 -1.57 
- added joint imu_joint: type fixed, parent base_link, child imu_link, origin xyz=0.0 0 -0.1 rpy=0 0 0
- added joint laser_joint: type fixed, parent base_link, child laser_link, origin xyz=0.103 0 -0.034 rpy=0 0 0
